File: PCB/3720-ST/3720-ST.kicad_sch (KiCad schematic)
At the start: 34 parts, among them J1 1546216-8, J10 1546216-8, J11 1546216-8, J12 1546216-8, J13 1546216-8, J14 1546216-8, J15 1546216-8, J16 1546216-8, J2 1546216-8, J3 1546216-8, J4 1546216-8, J5 1546216-8, J6 1546216-8, J7 1546216-8, J8 1546216-8, J9 1546216-8, U1 TMP275AID, U2 TMP275AID, U3 TMP275AID, U4 TMP275AID

Commit message: latest fixes and added via stitching
Connections:
- net 3V3 is gone; now on net +3V3: MUX2.73
- net SCLK is gone; now on net SCL: MUX2.74
Changed lines of the file:
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@@
-    (effects (font (size 1.27 1.27)) (justify right bottom))
-  )
-  (label "3V3" (at 213.36 109.22 180)
     (effects (font (size 1.27 1.27)) (justify right bottom))
   )
@@
     (effects (font (size 1.27 1.27)) (justify left bottom))
   )
-  (label "SCLK" (at 213.36 111.76 180)
+  (label "SCL" (at 213.36 111.76 180)
     (effects (font (size 1.27 1.27)) (justify right bottom))
   )
@@
     (pin "2")
   )
+  (symbol (lib_id "power:+3.3V") (at 213.36 109.22 270) (unit 1)
+    (in_bom yes) (on_board yes) (fields_autoplaced)
+    (property "Reference" "#PWR?" (id 0) (at 209.55 109.22 0)
+      (effects (font (size 1.27 1.27)) hide)
+    )
+    (property "Value" "+3.3V" (id 1) (at 216.535 109.6538 90)
+      (effects (font (size 1.27 1.27)) (justify left))
+    )
+    (property "Footprint" "" (id 2) (at 213.36 109.22 0)
+      (effects (font (size 1.27 1.27)) hide)
+    )
+    (property "Datasheet" "" (id 3) (at 213.36 109.22 0)
+      (effects (font (size 1.27 1.27)) hide)
+    )
+    (pin "1")
+  )
   (symbol (lib_id "Device:R_Small_US") (at 313.69 133.35 0) (unit 1)
     (in_bom yes) (on_board yes) (fields_autoplaced)
@@
       (reference "#PWR0123") (unit 1) (value "+3.3V") (footprint "")
     )
+    (path "/90838381-6e57-4a5b-98b5-d87b635f788a"
+      (reference "#PWR?") (unit 1) (value "+3.3V") (footprint "")
+    )
     (path "/cfa21871-4d6c-4070-a3cb-255462736cdf"
